File: SHT31_RS485.kicad_sch (KiCad schematic)
At the start: 33 parts, among them IC1 MP1584EN, J1 Connector, U1 STM32F030F4Px, U2 SHT31-DIS, U3 SP3485EN

Commit message: Add MP1584EN Diose.
Parts:
- added D2: SS34, Anh_Footprints:D_SMA, symbol Anh_Symbols:SS34
- added J2: ADC, Connector_JST:JST_GH_BM02B-GHS-TBT_1x02-1MP_P1.25mm_Vertical, symbol Connector:Conn_01x02_Pin
- J1: footprint Conn_Horizontal_2Layer:Conn_02x02_Horizontal_2Layer -> Anh_Footprints:Conn_02x02_Horizontal_2Layer
Connections:
- net GND: now also D2.2, J2.1 (Pin_1)
- net at C1.2, IC1.1 (SW), L1.1: now also D2.1
- net ADC: now reaches U1.6 (PA0)
- net ADC: now also J2.2 (Pin_2)
- no-connect marks 10 -> 9
Other:
- moved on the sheet: C3, C4, C5, L1, R7, R8
